Commit message: 251203_lidar_direction

File: src/rosmaster_description/urdf/ugv.urdf.xacro (robot description, xacro)
@@ -190,5 +190,6 @@
     <parent link="base_link"/>
     <child link="laser_link"/>
-    <origin xyz="${LIDAR_X} 0 ${LIDAR_Z}" rpy="0 0 ${PI}"/>
+    <!-- LIDAR를 전면을 바라보도록 yaw 회전을 0으로 설정 -->
+    <origin xyz="${LIDAR_X} 0 ${LIDAR_Z}" rpy="0 0 0"/>
   </joint>
   <joint name="imu_joint" type="fixed">

Commit message: 20251230_scan

File: src/rosmaster_description/urdf/ugv.urdf.xacro (robot description, xacro)
@@ -191,5 +191,5 @@
     <child link="laser_link"/>
     <!-- LIDAR 데이터가 실제 전면과 일치하도록 180도 회전 -->
-    <origin xyz="${LIDAR_X} 0 ${LIDAR_Z}" rpy="0 0 ${PI}"/>
+    <origin xyz="${LIDAR_X} 0 ${LIDAR_Z}" rpy="0 0 0"/>
   </joint>
   <joint name="imu_joint" type="fixed">

Commit message: 20251230_scan

File: src/rosmaster_description/urdf/ugv.urdf.xacro (robot description, xacro)
@@ -191,5 +191,5 @@
     <child link="laser_link"/>
     <!-- LIDAR 데이터가 실제 전면과 일치하도록 180도 회전 -->
-    <origin xyz="${LIDAR_X} 0 ${LIDAR_Z}" rpy="0 0 0"/>
+    <origin xyz="${LIDAR_X} 0 ${LIDAR_Z}" rpy="0 0 ${PI}"/>
   </joint>
   <joint name="imu_joint" type="fixed">

Commit message: 20251230_map

File: src/rosmaster_description/urdf/ugv.urdf.xacro (robot description, xacro)
@@ -7,6 +7,6 @@
   <xacro:property name="BASE_MASS"    value="20.0"/>
   <!-- 휠 파라미터 (rosmaster_base_node와 일치) -->
-  <xacro:property name="WHEEL_RADIUS" value="0.095"/>
-  <xacro:property name="WHEEL_WIDTH"  value="0.095"/>
+  <xacro:property name="WHEEL_RADIUS" value="0.097"/>
+  <xacro:property name="WHEEL_WIDTH"  value="0.097"/>
   <xacro:property name="TRACK_WIDTH"  value="0.482"/>   <!-- 좌/우 바퀴 간 거리 -->
   <xacro:property name="WHEELBASE"    value="0.255"/>   <!-- 전/후 바퀴 간 거리 -->

Commit message: 20251230_map

File: src/rosmaster_description/urdf/ugv.urdf.xacro (robot description, xacro)
@@ -9,5 +9,5 @@
   <xacro:property name="WHEEL_RADIUS" value="0.097"/>
   <xacro:property name="WHEEL_WIDTH"  value="0.097"/>
-  <xacro:property name="TRACK_WIDTH"  value="0.482"/>   <!-- 좌/우 바퀴 간 거리 -->
+  <xacro:property name="TRACK_WIDTH"  value="0.483"/>   <!-- 좌/우 바퀴 간 거리 -->
   <xacro:property name="WHEELBASE"    value="0.255"/>   <!-- 전/후 바퀴 간 거리 -->
   <xacro:property name="WHEEL_MASS"   value="0.1"/>
